Commit message: blubb

File: model/test_3dof.urdf (robot description, URDF)
Before this commit: robot lbr_iiwa, 5 links, 4 joints
Joints:
- joint joint1: limit lower=-3.14159265358979323846 upper=3.14159265358979323846 effort=150 velocity=10 -> lower=-3.14159265358979323846 upper=3.14159265358979323846 effort=150 velocity=15
- joint joint2: limit lower=-3.14159265358979323846 upper=3.14159265358979323846 effort=70 velocity=10 -> lower=-3.14159265358979323846 upper=3.14159265358979323846 effort=70 velocity=15
- joint joint3: limit lower=-3.14159265358979323846 upper=3.14159265358979323846 effort=60 velocity=10 -> lower=-3.14159265358979323846 upper=3.14159265358979323846 effort=60 velocity=15

Commit message: Added sensors

File: model/test_3dof.urdf (robot description, URDF)
Before this commit: robot lbr_iiwa, 5 links, 4 joints
Joints:
- joint joint1: origin xyz=0 0 5 rpy=0 0 0 -> xyz=0 0 8 rpy=0 0 0
